File: kicad/TTl-logic-probe/TTl-logic-probe.kicad_sch (KiCad schematic)
At the start: 25 parts, among them J1 Conn_01x01_Pin, J2 Conn_01x02_Pin, U1 74HC04, U2 74HC00, U3 74HC93

Commit message: Updated README.md
Parts:
- U1: value 74HC04 -> 74LS04
- U2: value 74HC00 -> 74LS00
- U3: value 74HC93 -> 74LS93
Other:
- moved on the sheet: U2C, U2D
Changed lines of the file:
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@@
   (junction (at 76.2 67.945) (diameter 0) (color 0 0 0 0)
   )
-  (junction (at 74.93 86.36) (diameter 0) (color 0 0 0 0)
+  (junction (at 86.36 86.995) (diameter 0) (color 0 0 0 0)
   )
   (junction (at 189.23 76.835) (diameter 0) (color 0 0 0 0)
@@
   (junction (at 189.23 69.215) (diameter 0) (color 0 0 0 0)
   )
-  (junction (at 92.71 86.36) (diameter 0) (color 0 0 0 0)
+  (junction (at 104.14 86.995) (diameter 0) (color 0 0 0 0)
   )
   (junction (at 197.485 124.46) (diameter 0) (color 0 0 0 0)
   )
-  (junction (at 67.945 73.025) (diameter 0) (color 0 0 0 0)
+  (junction (at 76.2 73.025) (diameter 0) (color 0 0 0 0)
   )
   (junction (at 37.465 67.945) (diameter 0) (color 0 0 0 0)
@@
     (stroke (width 0) (type default))
   )
-  (wire (pts (xy 74.93 86.36) (xy 74.93 88.9))
-    (stroke (width 0) (type default))
-  )
-  (wire (pts (xy 74.93 86.36) (xy 67.945 86.36))
+  (wire (pts (xy 86.36 86.995) (xy 86.36 89.535))
+    (stroke (width 0) (type default))
+  )
+  (wire (pts (xy 86.36 86.995) (xy 76.2 86.995))
     (stroke (width 0) (type default))
   )
@@
     (stroke (width 0) (type default))
   )
-  (wire (pts (xy 92.71 86.36) (xy 92.71 88.9))
-    (stroke (width 0) (type default))
-  )
-  (wire (pts (xy 107.95 86.36) (xy 127.635 86.36))
+  (wire (pts (xy 104.14 86.995) (xy 104.14 89.535))
+    (stroke (width 0) (type default))
+  )
+  (wire (pts (xy 119.38 86.995) (xy 127.635 86.995))
     (stroke (width 0) (type default))
   )
@@
     (stroke (width 0) (type default))
   )
-  (wire (pts (xy 90.17 86.36) (xy 92.71 86.36))
+  (wire (pts (xy 101.6 86.995) (xy 104.14 86.995))
     (stroke (width 0) (type default))
   )
@@
     (stroke (width 0) (type default))
   )
-  (wire (pts (xy 92.71 83.82) (xy 92.71 86.36))
+  (wire (pts (xy 104.14 84.455) (xy 104.14 86.995))
     (stroke (width 0) (type default))
   )
@@
     (stroke (width 0) (type default))
   )
+  (wire (pts (xy 76.2 73.025) (xy 86.36 73.025))
+    (stroke (width 0) (type default))
+  )
   (wire (pts (xy 261.62 66.04) (xy 261.62 78.74))
     (stroke (width 0) (type default))
   )
-  (wire (pts (xy 74.93 83.82) (xy 74.93 86.36))
+  (wire (pts (xy 86.36 84.455) (xy 86.36 86.995))
     (stroke (width 0) (type default))
   )
@@
     (stroke (width 0) (type default))
   )
-  (wire (pts (xy 37.465 73.025) (xy 67.945 73.025))
+  (wire (pts (xy 37.465 73.025) (xy 76.2 73.025))
     (stroke (width 0) (type default))
   )
@@
     (stroke (width 0) (type default))
   )
-  (wire (pts (xy 127.635 84.455) (xy 127.635 86.36))
-    (stroke (width 0) (type default))
-  )
-  (wire (pts (xy 67.945 73.025) (xy 86.36 73.025))
-    (stroke (width 0) (type default))
-  )
-  (wire (pts (xy 67.945 86.36) (xy 67.945 73.025))
+  (wire (pts (xy 127.635 84.455) (xy 127.635 86.995))
+    (stroke (width 0) (type default))
+  )
+  (wire (pts (xy 76.2 86.995) (xy 76.2 73.025))
     (stroke (width 0) (type default))
   )
@@
       (effects (font (size 1.27 1.27)))
     )
-    (property "Value" "74HC00" (at 93.9717 64.77 0)
+    (property "Value" "74LS00" (at 93.9717 64.77 0)
       (effects (font (size 1.27 1.27)))
     )
@@
     )
   )
-  (symbol (lib_id "74xx:74HC00") (at 100.33 86.36 0) (unit 4)
-    (in_bom yes) (on_board yes) (dnp no) (fields_autoplaced)
-    (property "Reference" "U2" (at 100.3217 77.47 0)
-      (effects (font (size 1.27 1.27)))
-    )
-    (property "Value" "74HC00" (at 100.3217 80.01 0)
-      (effects (font (size 1.27 1.27)))
-    )
-    (property "Footprint" "Package_DIP:DIP-14_W7.62mm" (at 100.33 86.36 0)
-      (effects (font (size 1.27 1.27)) hide)
-    )
-    (property "Datasheet" "http://www.ti.com/lit/gpn/sn74hc00" (at 100.33 86.36 0)
-      (effects (font (size 1.27 1.27)) hide)
-    )
-    (property "Mfr. No" "74HC00" (at 100.33 86.36 0)
+  (symbol (lib_id "74xx:74HC00") (at 111.76 86.995 0) (unit 4)
+    (in_bom yes) (on_board yes) (dnp no) (fields_autoplaced)
+    (property "Reference" "U2" (at 111.7517 78.105 0)
+      (effects (font (size 1.27 1.27)))
+    )
+    (property "Value" "74LS00" (at 111.7517 80.645 0)
+      (effects (font (size 1.27 1.27)))
+    )
+    (property "Footprint" "Package_DIP:DIP-14_W7.62mm" (at 111.76 86.995 0)
+      (effects (font (size 1.27 1.27)) hide)
+    )
+    (property "Datasheet" "http://www.ti.com/lit/gpn/sn74hc00" (at 111.76 86.995 0)
+      (effects (font (size 1.27 1.27)) hide)
+    )
+    (property "Mfr. No" "74HC00" (at 111.76 86.995 0)
       (effects (font (size 1.27 1.27)) hide)
     )
@@
       (effects (font (size 1.27 1.27)))
     )
-    (property "Value" "74HC00" (at 75.565 116.84 0)
+    (property "Value" "74LS00" (at 75.565 116.84 0)
       (effects (font (size 1.27 1.27)))
     )
@@
       (effects (font (size 1.27 1.27)))
     )
-    (property "Value" "74HC04" (at 92.71 116.205 0)
+    (property "Value" "74LS04" (at 92.71 116.205 0)
       (effects (font (size 1.27 1.27)))
     )
@@
       (effects (font (size 1.27 1.27)))
     )
-    (property "Value" "74HC04" (at 179.705 84.455 0)
+    (property "Value" "74LS04" (at 179.705 84.455 0)
       (effects (font (size 1.27 1.27)))
     )
@@
       (effects (font (size 1.27 1.27)))
     )
-    (property "Value" "74HC04" (at 233.045 99.695 0)
+    (property "Value" "74LS04" (at 233.045 99.695 0)
       (effects (font (size 1.27 1.27)))
     )
@@
       (effects (font (size 1.27 1.27)))
     )
-    (property "Value" "74HC00" (at 62.8567 62.23 0)
+    (property "Value" "74LS00" (at 62.8567 62.23 0)
       (effects (font (size 1.27 1.27)))
     )
@@
       (effects (font (size 1.27 1.27)) (justify left))
     )
-    (property "Value" "74HC93" (at 204.1241 63.5 0)
+    (property "Value" "74LS93" (at 204.1241 63.5 0)
       (effects (font (size 1.27 1.27)) (justify left))
     )
@@
       (effects (font (size 1.27 1.27)))
     )
-    (property "Value" "74HC04" (at 158.115 76.835 0)
+    (property "Value" "74LS04" (at 158.115 76.835 0)
       (effects (font (size 1.27 1.27)))
     )
@@
       (effects (font (size 1.27 1.27)))
     )
-    (property "Value" "74HC04" (at 232.41 86.36 0)
+    (property "Value" "74LS04" (at 232.41 86.36 0)
       (effects (font (size 1.27 1.27)))
     )
@@
     )
   )
-  (symbol (lib_id "74xx:74HC00") (at 82.55 86.36 0) (unit 3)
-    (in_bom yes) (on_board yes) (dnp no) (fields_autoplaced)
-    (property "Reference" "U2" (at 82.5417 78.105 0)
-      (effects (font (size 1.27 1.27)))
-    )
-    (property "Value" "74HC00" (at 82.5417 80.645 0)
-      (effects (font (size 1.27 1.27)))
-    )
-    (property "Footprint" "Package_DIP:DIP-14_W7.62mm" (at 82.55 86.36 0)
-      (effects (font (size 1.27 1.27)) hide)
-    )
-    (property "Datasheet" "http://www.ti.com/lit/gpn/sn74hc00" (at 82.55 86.36 0)
-      (effects (font (size 1.27 1.27)) hide)
-    )
-    (property "Mfr. No" "74HC00" (at 82.55 86.36 0)
+  (symbol (lib_id "74xx:74HC00") (at 93.98 86.995 0) (unit 3)
+    (in_bom yes) (on_board yes) (dnp no) (fields_autoplaced)
+    (property "Reference" "U2" (at 93.9717 78.74 0)
+      (effects (font (size 1.27 1.27)))
+    )
+    (property "Value" "74LS00" (at 93.9717 81.28 0)
+      (effects (font (size 1.27 1.27)))
+    )
+    (property "Footprint" "Package_DIP:DIP-14_W7.62mm" (at 93.98 86.995 0)
+      (effects (font (size 1.27 1.27)) hide)
+    )
+    (property "Datasheet" "http://www.ti.com/lit/gpn/sn74hc00" (at 93.98 86.995 0)
+      (effects (font (size 1.27 1.27)) hide)
+    )
+    (property "Mfr. No" "74HC00" (at 93.98 86.995 0)
       (effects (font (size 1.27 1.27)) hide)
     )
@@
       (effects (font (size 1.27 1.27)))
     )
-    (property "Value" "74HC04" (at 232.41 73.66 0)
+    (property "Value" "74LS04" (at 232.41 73.66 0)
       (effects (font (size 1.27 1.27)))
     )
@@
       (effects (font (size 1.27 1.27)))
     )
-    (property "Value" "74HC04" (at 232.41 60.96 0)
-      (effects (font (size 1.27 1.27)))
-    )
+    (property "Value" "74LS04" (at 232.41 60.96 0)
+      (effects (font (size 1.27 1.27)))
+    )
